File: PCA9535/PCA9535.kicad_sch (KiCad schematic)
At the start: 5 parts

Commit message: progress
Parts:
- removed J? (x2): Conn_02x08_Counter_Clockwise, symbol Connector_Generic:Conn_02x08_Counter_Clockwise
- added H1, H2, H3, H4: MountingHole, MountingHole:MountingHole_2.5mm, symbol Mechanical:MountingHole
- added J3, J6: Conn_02x05_Odd_Even, symbol Connector_Generic:Conn_02x05_Odd_Even
- added J4: Conn_01x01, Connector_PinHeader_2.54mm:PinHeader_1x01_P2.54mm_Vertical, symbol Connector_Generic:Conn_01x01
- added J5: Conn_01x10, Connector_PinHeader_2.54mm:PinHeader_1x10_P2.54mm_Vertical, symbol Connector_Generic:Conn_01x10
- added R1, R2, R3: R, Resistor_SMD:R_0805_2012Metric_Pad1.20x1.40mm_HandSolder, symbol Device:R
- J1, J2: renamed from J?; footprint (none) -> Connector_JST:JST_SH_BM04B-SRSS-TB_1x04-1MP_P1.00mm_Vertical
- U1: renamed from U?; footprint DB24_TEX -> ul_PCA9535DBR:PCA9535DBR
Connections:
- net GND: now reaches J2.1 (Pin_1)
- net GND: now also J1.1 (Pin_1), U1.12 (GND), J5.10 (Pin_10), J6.10 (Pin_10)
- net +3.3V: now reaches J2.2 (Pin_2)
- net +3.3V: now also J1.2 (Pin_2), U1.24 (VCC), J5.9 (Pin_9), J6.9 (Pin_9), R1.1, R2.1, R3.1
- net SDA: now reaches J2.3 (Pin_3)
- net SDA: now also J1.3 (Pin_3), U1.23 (SDA), R2.2
- net SCL: now reaches J2.4 (Pin_4)
- net SCL: now also J1.4 (Pin_4), U1.22 (SCL), R1.2
- net INT: now reaches U1.1 (*INT)
- net INT: now also J4.1 (Pin_1), R3.2
- net P06: now reaches U1.10 (P06)
- net P06: now also J5.7 (Pin_7)
- net P07: now reaches U1.11 (P07)
- net P07: now also J5.8 (Pin_8)
- net P10: now reaches U1.13 (P10)
- net P10: now also J6.1 (Pin_1)
- net P11: now reaches U1.14 (P11)
- net P11: now also J6.3 (Pin_3)
- net P12: now reaches U1.15 (P12)
- net P12: now also J6.5 (Pin_5)
- net P13: now reaches U1.16 (P13)
- net P13: now also J6.7 (Pin_7)
- net P14: now reaches U1.17 (P14)
- net P14: now also J6.2 (Pin_2)
- net P15: now reaches U1.18 (P15)
- net P15: now also J6.4 (Pin_4)
- net P16: now reaches U1.19 (P16)
- net P16: now also J6.6 (Pin_6)
- net A1: now reaches U1.2 (A1)
- net P17: now reaches U1.20 (P17)
- net P17: now also J6.8 (Pin_8)
- net A0: now reaches U1.21 (A0)
- net A2: now reaches U1.3 (A2)
- net P00: now reaches U1.4 (P00)
- net P00: now also J5.1 (Pin_1)
- net P01: now reaches U1.5 (P01)
- net P01: now also J5.2 (Pin_2)
- net P02: now reaches U1.6 (P02)
- net P02: now also J5.3 (Pin_3)
- net P03: now reaches U1.7 (P03)
- net P03: now also J5.4 (Pin_4)
- net P04: now reaches U1.8 (P04)
- net P04: now also J5.5 (Pin_5)
- net P05: now reaches U1.9 (P05)
- net P05: now also J5.6 (Pin_6)
Other:
- moved on the sheet: J2
