File: PCA9535/PCA9535.kicad_pcb (KiCad board)
At the start: 2 copper layers, 25 x 25 mm, 13 parts, among them J1 Conn_01x04, J2 Conn_01x04, J3 Conn_01x10, J4 Conn_01x01, J5 Conn_01x10, U1 PCA9535DBR

Commit message: Updating GPIO expansion board
Parts:
- removed J5: Conn_01x10, Connector_PinHeader_2.54mm:PinHeader_1x10_P2.54mm_Vertical
- added J6: Conn_02x05_Odd_Even, Connector_PinHeader_2.54mm:PinHeader_2x05_P2.54mm_Vertical, F.Cu at (140.0, 87.0)
- J3: value Conn_01x10 -> Conn_02x05_Odd_Even; footprint Connector_PinHeader_2.54mm:PinHeader_1x10_P2.54mm_Vertical -> Connector_PinHeader_2.54mm:PinHeader_2x05_P2.54mm_Vertical
- R1, R2, R3: value R -> 4.7k
- moved J3 16.4 mm to (118.5, 77.0), turned to 0 degrees
- moved J4 10.0 mm to (129.0, 77.0)
- moved R1 5.70 mm to (133.0, 78.0)
- moved R2 5.70 mm to (133.0, 76.0)
- moved R3 2.50 mm to (125.0, 77.0), turned to 0 degrees
- moved U1 0.50 mm to (128.4, 84.0)
Connections:
- J3 pad 1: P10 -> P00
- J3 pad 2: P11 -> P04
- J3 pad 3: P12 -> P01
- J3 pad 4: P13 -> P05
- J3 pad 5: P14 -> P02
- J3 pad 6: P15 -> P06
- J3 pad 7: P16 -> P03
- J3 pad 8: P17 -> P07
Routing:
- net +3.3V: track 37.3 -> 54.2 mm
- net P12: track 0.00 -> 12.3 mm, vias 0 -> 1
- net P13: track 0.00 -> 12.0 mm, vias 0 -> 1
- net P11: track 0.00 -> 9.55 mm, vias 0 -> 1
- net P10: track 0.00 -> 8.70 mm
- net SCL: track 23.7 -> 15.1 mm
- net P04: track 17.1 -> 10.1 mm, vias 1 -> 0
- net P17: track 0.00 -> 6.90 mm
- net P14: track 0.00 -> 6.27 mm
- net P16: track 0.00 -> 6.12 mm
- net P15: track 0.00 -> 5.48 mm
- net P06: track 1.83 -> 6.33 mm, vias 1 -> 0
- net P02: track 17.0 -> 12.9 mm
- net SDA: track 21.0 -> 18.4 mm, vias 3 -> 0
- net P00: track 15.5 -> 13.3 mm, vias 0 -> 1
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Other:
- board text added: "3v3"
- board text added: "Designed by Fortinbra fortinbra@becauseimclever.com"
- board text added: "GND"

Commit message: Figured out solder jumpers, kinda
Parts:
- added JP1: SolderJumper_3_Open, Jumper:SolderJumper-3_P1.3mm_Open_Pad1.0x1.5mm, B.Cu at (130.5, 84.5)
- added JP2: SolderJumper_3_Open, Jumper:SolderJumper-3_P1.3mm_Open_Pad1.0x1.5mm, B.Cu at (130.5, 88.5)
- added JP3: SolderJumper_3_Open, Jumper:SolderJumper-3_P1.3mm_Open_Pad1.0x1.5mm, B.Cu at (130.5, 92.5)
Changed lines of the file:
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@@
     (pad "" np_thru_hole circle (at 0 0) (size 2.5 2.5) (drill 2.5) (layers *.Cu *.Mask))
+  )
+  (footprint "Jumper:SolderJumper-3_P1.3mm_Open_Pad1.0x1.5mm" (layer "B.Cu")
+    (at 130.5 84.5 180)
+    (descr "SMD Solder 3-pad Jumper, 1x1.5mm Pads, 0.3mm gap, open")
+    (tags "solder jumper open")
+    (property "Sheetfile" "PCA9535.kicad_sch")
+    (property "Sheetname" "")
+    (attr exclude_from_pos_files)
+    (fp_text reference "JP1" (at 0 1.8) (layer "B.SilkS")
+      (effects (font (size 1 1) (thickness 0.15)) (justify mirror))
+    )
+    (fp_text value "SolderJumper_3_Open" (at 0 -2) (layer "B.Fab")
+      (effects (font (size 1 1) (thickness 0.15)) (justify mirror))
+    )
+    (fp_line (start 2.05 -1) (end -2.05 -1) (layer "B.SilkS") (width 0.12))
+    (fp_line (start -1.3 -1.2) (end -1 -1.5) (layer "B.SilkS") (width 0.12))
+    (fp_line (start -2.05 1) (end 2.05 1) (layer "B.SilkS") (width 0.12))
+    (fp_line (start -2.05 -1) (end -2.05 1) (layer "B.SilkS") (width 0.12))
+    (fp_line (start 2.05 1) (end 2.05 -1) (layer "B.SilkS") (width 0.12))
+    (fp_line (start -1.3 -1.2) (end -1.6 -1.5) (layer "B.SilkS") (width 0.12))
+    (fp_line (start -1.6 -1.5) (end -1 -1.5) (layer "B.SilkS") (width 0.12))
+    (fp_line (start -2.3 1.25) (end -2.3 -1.25) (layer "B.CrtYd") (width 0.05))
+    (fp_line (start -2.3 1.25) (end 2.3 1.25) (layer "B.CrtYd") (width 0.05))
+    (fp_line (start 2.3 -1.25) (end -2.3 -1.25) (layer "B.CrtYd") (width 0.05))
+    (fp_line (start 2.3 -1.25) (end 2.3 1.25) (layer "B.CrtYd") (width 0.05))
+    (pad "1" smd rect (at -1.3 0 180) (size 1 1.5) (layers "B.Cu" "B.Mask")
+      (net 1 "+3.3V") (pinfunction "A") (pintype "passive"))
+    (pad "2" smd rect (at 0 0 180) (size 1 1.5) (layers "B.Cu" "B.Mask")
+      (net 24 "A0") (pinfunction "C") (pintype "passive"))
+    (pad "3" smd rect (at 1.3 0 180) (size 1 1.5) (layers "B.Cu" "B.Mask")
+      (net 4 "GND") (pinfunction "B") (pintype "passive"))
+  )
+  (footprint "Jumper:SolderJumper-3_P1.3mm_Open_Pad1.0x1.5mm" (layer "B.Cu")
+    (at 130.5 88.5 180)
+    (descr "SMD Solder 3-pad Jumper, 1x1.5mm Pads, 0.3mm gap, open")
+    (tags "solder jumper open")
+    (property "Sheetfile" "PCA9535.kicad_sch")
+    (property "Sheetname" "")
+    (attr exclude_from_pos_files)
+    (fp_text reference "JP2" (at 0 1.8) (layer "B.SilkS")
+      (effects (font (size 1 1) (thickness 0.15)) (justify mirror))
+    )
+    (fp_text value "SolderJumper_3_Open" (at 0 -2) (layer "B.Fab")
+      (effects (font (size 1 1) (thickness 0.15)) (justify mirror))
+    )
+    (fp_line (start -1.3 -1.2) (end -1 -1.5) (layer "B.SilkS") (width 0.12))
+    (fp_line (start -2.05 1) (end 2.05 1) (layer "B.SilkS") (width 0.12))
+    (fp_line (start -1.6 -1.5) (end -1 -1.5) (layer "B.SilkS") (width 0.12))
+    (fp_line (start -1.3 -1.2) (end -1.6 -1.5) (layer "B.SilkS") (width 0.12))
+    (fp_line (start 2.05 -1) (end -2.05 -1) (layer "B.SilkS") (width 0.12))
+    (fp_line (start -2.05 -1) (end -2.05 1) (layer "B.SilkS") (width 0.12))
+    (fp_line (start 2.05 1) (end 2.05 -1) (layer "B.SilkS") (width 0.12))
+    (fp_line (start -2.3 1.25) (end 2.3 1.25) (layer "B.CrtYd") (width 0.05))
+    (fp_line (start -2.3 1.25) (end -2.3 -1.25) (layer "B.CrtYd") (width 0.05))
+    (fp_line (start 2.3 -1.25) (end 2.3 1.25) (layer "B.CrtYd") (width 0.05))
+    (fp_line (start 2.3 -1.25) (end -2.3 -1.25) (layer "B.CrtYd") (width 0.05))
+    (pad "1" smd rect (at -1.3 0 180) (size 1 1.5) (layers "B.Cu" "B.Mask")
+      (net 1 "+3.3V") (pinfunction "A") (pintype "passive"))
+    (pad "2" smd rect (at 0 0 180) (size 1 1.5) (layers "B.Cu" "B.Mask")
+      (net 21 "A1") (pinfunction "C") (pintype "passive"))
+    (pad "3" smd rect (at 1.3 0 180) (size 1 1.5) (layers "B.Cu" "B.Mask")
+      (net 4 "GND") (pinfunction "B") (pintype "passive"))
+  )
+  (footprint "Jumper:SolderJumper-3_P1.3mm_Open_Pad1.0x1.5mm" (layer "B.Cu")
+    (at 130.5 92.5 180)
+    (descr "SMD Solder 3-pad Jumper, 1x1.5mm Pads, 0.3mm gap, open")
+    (tags "solder jumper open")
+    (property "Sheetfile" "PCA9535.kicad_sch")
+    (property "Sheetname" "")
+    (attr exclude_from_pos_files)
+    (fp_text reference "JP3" (at 0 1.8) (layer "B.SilkS")
+      (effects (font (size 1 1) (thickness 0.15)) (justify mirror))
+    )
+    (fp_text value "SolderJumper_3_Open" (at 0 -2) (layer "B.Fab") hide
+      (effects (font (size 1 1) (thickness 0.15)) (justify mirror))
+    )
+    (fp_line (start -2.05 -1) (end -2.05 1) (layer "B.SilkS") (width 0.12))
+    (fp_line (start -2.05 1) (end 2.05 1) (layer "B.SilkS") (width 0.12))
+    (fp_line (start -1.3 -1.2) (end -1.6 -1.5) (layer "B.SilkS") (width 0.12))
+    (fp_line (start -1.3 -1.2) (end -1 -1.5) (layer "B.SilkS") (width 0.12))
+    (fp_line (start 2.05 1) (end 2.05 -1) (layer "B.SilkS") (width 0.12))
+    (fp_line (start -1.6 -1.5) (end -1 -1.5) (layer "B.SilkS") (width 0.12))
+    (fp_line (start 2.05 -1) (end -2.05 -1) (layer "B.SilkS") (width 0.12))
+    (fp_line (start -2.3 1.25) (end 2.3 1.25) (layer "B.CrtYd") (width 0.05))
+    (fp_line (start 2.3 -1.25) (end -2.3 -1.25) (layer "B.CrtYd") (width 0.05))
+    (fp_line (start 2.3 -1.25) (end 2.3 1.25) (layer "B.CrtYd") (width 0.05))
+    (fp_line (start -2.3 1.25) (end -2.3 -1.25) (layer "B.CrtYd") (width 0.05))
+    (pad "1" smd rect (at -1.3 0 180) (size 1 1.5) (layers "B.Cu" "B.Mask")
+      (net 1 "+3.3V") (pinfunction "A") (pintype "passive"))
+    (pad "2" smd rect (at 0 0 180) (size 1 1.5) (layers "B.Cu" "B.Mask")
+      (net 22 "A2") (pinfunction "C") (pintype "passive"))
+    (pad "3" smd rect (at 1.3 0 180) (size 1 1.5) (layers "B.Cu" "B.Mask")
+      (net 4 "GND") (pinfunction "B") (pintype "passive"))
   )
   (gr_rect (start 116.5 69.5) (end 141.5 94.5) (layer "Edge.Cuts") (width 0.1) (fill none))

Commit message: sync
Routing:
- net +3.3V: track 54.2 -> 90.3 mm
- net A2: track 0.00 -> 14.9 mm, vias 0 -> 1
- net A1: track 0.00 -> 12.1 mm, vias 0 -> 1
- net SCL: track 15.1 -> 18.5 mm, vias 3 -> 4
- net A0: track 0.00 -> 2.94 mm, vias 0 -> 1
- net P00: track 13.3 -> 14.3 mm
- net P01: track 12.6 -> 13.3 mm
- net GND: vias 0 -> 3
Changed lines of the file:
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@@
   (segment (start 134 78.428801) (end 134 78) (width 0.25) (layer "F.Cu") (net 1))
   (segment (start 124.5 72.878249) (end 125.153249 72.225) (width 0.25) (layer "F.Cu") (net 1))
+  (segment (start 136.836442 78.015) (end 131.8 83.051442) (width 0.25) (layer "B.Cu") (net 1))
+  (segment (start 138.825 78.015) (end 136.836442 78.015) (width 0.25) (layer "B.Cu") (net 1))
+  (segment (start 140 76.84) (end 138.825 78.015) (width 0.25) (layer "B.Cu") (net 1))
+  (segment (start 131.8 92.5) (end 131.8 88.5) (width 0.25) (layer "B.Cu") (net 1))
+  (segment (start 131.8 83.051442) (end 131.8 84.5) (width 0.25) (layer "B.Cu") (net 1))
+  (segment (start 131.325 91.425) (end 131.8 91.9) (width 0.25) (layer "B.Cu") (net 1))
+  (segment (start 131.8 88.5) (end 131.8 84.5) (width 0.25) (layer "B.Cu") (net 1))
+  (segment (start 118.5 87.16) (end 122.765 91.425) (width 0.25) (layer "B.Cu") (net 1))
+  (segment (start 131.8 91.9) (end 131.8 92.5) (width 0.25) (layer "B.Cu") (net 1))
+  (segment (start 122.765 91.425) (end 131.325 91.425) (width 0.25) (layer "B.Cu") (net 1))
   (segment (start 133.5 74.5) (end 132 76) (width 0.25) (layer "F.Cu") (net 2))
   (segment (start 125.5 73.325) (end 125.5 75) (width 0.25) (layer "F.Cu") (net 2))
@@
   (segment (start 126.5 73.325) (end 128.325 73.325) (width 0.25) (layer "F.Cu") (net 3))
   (segment (start 130 81.5) (end 130.287002 81.787002) (width 0.25) (layer "F.Cu") (net 3))
+  (via (at 134.5 73.5) (size 0.8) (drill 0.4) (layers "F.Cu" "B.Cu") (net 3))
   (via (at 132 78) (size 0.8) (drill 0.4) (layers "F.Cu" "B.Cu") (net 3))
   (via (at 128.5 73.5) (size 0.8) (drill 0.4) (layers "F.Cu" "B.Cu") (net 3))
@@
   (segment (start 132 78) (end 130 80) (width 0.25) (layer "B.Cu") (net 3))
   (segment (start 130 80) (end 130 81.5) (width 0.25) (layer "B.Cu") (net 3))
+  (segment (start 132.5 75.5) (end 132 75.5) (width 0.25) (layer "B.Cu") (net 3))
+  (segment (start 134.5 73.5) (end 132.5 75.5) (width 0.25) (layer "B.Cu") (net 3))
   (segment (start 132 75.5) (end 132 78) (width 0.25) (layer "B.Cu") (net 3))
   (segment (start 128.5 73.5) (end 130 73.5) (width 0.25) (layer "B.Cu") (net 3))
   (segment (start 130 73.5) (end 132 75.5) (width 0.25) (layer "B.Cu") (net 3))
-  (segment (start 125.672501 82.327499) (end 126.536898 81.463102) (width 0.25) (layer "F.Cu") (net 5))
-  (segment (start 124.7869 82.327499) (end 125.672501 82.327499) (width 0.25) (layer "F.Cu") (net 5))
-  (via (at 126.536898 81.463102) (size 0.8) (drill 0.4) (layers "F.Cu" "B.Cu") (net 5))
+  (via (at 127.5 92.5) (size 0.8) (drill 0.4) (layers "F.Cu" "B.Cu") (free) (net 4))
+  (via (at 131.5 73.5) (size 0.8) (drill 0.4) (layers "F.Cu" "B.Cu") (net 4))
+  (via (at 123.5 73.5) (size 0.8) (drill 0.4) (layers "F.Cu" "B.Cu") (net 4))
+  (segment (start 127.038534 81.96474) (end 126.675775 82.327499) (width 0.25) (layer "F.Cu") (net 5))
+  (segment (start 126.675775 82.327499) (end 124.7869 82.327499) (width 0.25) (layer "F.Cu") (net 5))
+  (via (at 127.038534 81.96474) (size 0.8) (drill 0.4) (layers "F.Cu" "B.Cu") (net 5))
+  (segment (start 122.573796 76.872095) (end 121.526701 75.825) (width 0.25) (layer "B.Cu") (net 5))
   (segment (start 122.573796 77.5) (end 122.573796 76.872095) (width 0.25) (layer "B.Cu") (net 5))
+  (segment (start 127.038534 81.96474) (end 122.573796 77.5) (width 0.25) (layer "B.Cu") (net 5))
+  (segment (start 119.675 75.825) (end 118.5 77) (width 0.25) (layer "B.Cu") (net 5))
   (segment (start 121.526701 75.825) (end 119.675 75.825) (width 0.25) (layer "B.Cu") (net 5))
-  (segment (start 119.675 75.825) (end 118.5 77) (width 0.25) (layer "B.Cu") (net 5))
-  (segment (start 126.536898 81.463102) (end 122.573796 77.5) (width 0.25) (layer "B.Cu") (net 5))
-  (segment (start 122.573796 76.872095) (end 121.526701 75.825) (width 0.25) (layer "B.Cu") (net 5))
-  (segment (start 126.425502 82.977498) (end 126.726098 82.676902) (width 0.25) (layer "F.Cu") (net 6))
-  (segment (start 124.7869 82.977498) (end 126.425502 82.977498) (width 0.25) (layer "F.Cu") (net 6))
-  (via (at 126.726098 82.676902) (size 0.8) (drill 0.4) (layers "F.Cu" "B.Cu") (net 6))
+  (segment (start 127.084386 83.03519) (end 127.026694 82.977498) (width 0.25) (layer "F.Cu") (net 6))
+  (segment (start 127.026694 82.977498) (end 124.7869 82.977498) (width 0.25) (layer "F.Cu") (net 6))
+  (via (at 127.084386 83.03519) (size 0.8) (drill 0.4) (layers "F.Cu" "B.Cu") (net 6))
+  (segment (start 119.675 78.365) (end 118.5 79.54) (width 0.25) (layer "B.Cu") (net 6))
+  (segment (start 127.084386 83.03519) (end 122.414196 78.365) (width 0.25) (layer "B.Cu") (net 6))
   (segment (start 122.414196 78.365) (end 119.675 78.365) (width 0.25) (layer "B.Cu") (net 6))
-  (segment (start 126.726098 82.676902) (end 122.414196 78.365) (width 0.25) (layer "B.Cu") (net 6))
-  (segment (start 119.675 78.365) (end 118.5 79.54) (width 0.25) (layer "B.Cu") (net 6))
-  (segment (start 127.041009 83.627499) (end 124.7869 83.627499) (width 0.25) (layer "F.Cu") (net 7))
-  (segment (start 127.206755 83.793245) (end 127.041009 83.627499) (width 0.25) (layer "F.Cu") (net 7))
-  (via (at 127.206755 83.793245) (size 0.8) (drill 0.4) (layers "F.Cu" "B.Cu") (net 7))
+  (segment (start 126.825205 84.054883) (end 126.397821 83.627499) (width 0.25) (layer "F.Cu") (net 7))
+  (segment (start 126.397821 83.627499) (end 124.7869 83.627499) (width 0.25) (layer "F.Cu") (net 7))
+  (via (at 126.825205 84.054883) (size 0.8) (drill 0.4) (layers "F.Cu" "B.Cu") (net 7))
+  (segment (start 126.825205 83.800607) (end 123.929598 80.905) (width 0.25) (layer "B.Cu") (net 7))
   (segment (start 123.929598 80.905) (end 119.675 80.905) (width 0.25) (layer "B.Cu") (net 7))
-  (segment (start 126.817843 83.793245) (end 123.929598 80.905) (width 0.25) (layer "B.Cu") (net 7))
-  (segment (start 127.206755 83.793245) (end 126.817843 83.793245) (width 0.25) (layer "B.Cu") (net 7))
+  (segment (start 126.825205 84.054883) (end 126.825205 83.800607) (width 0.25) (layer "B.Cu") (net 7))
   (segment (start 119.675 80.905) (end 118.5 82.08) (width 0.25) (layer "B.Cu") (net 7))
-  (segment (start 124.7869 84.277498) (end 126.277498 84.277498) (width 0.25) (layer "F.Cu") (net 8))
-  (segment (start 126.277498 84.277498) (end 126.5 84.5) (width 0.25) (layer "F.Cu") (net 8))
-  (via (at 126.5 84.5) (size 0.8) (drill 0.4) (layers "F.Cu" "B.Cu") (net 8))
+  (segment (start 126.5 85) (end 125.777498 84.277498) (width 0.25) (layer "F.Cu") (net 8))
+  (segment (start 125.777498 84.277498) (end 124.7869 84.277498) (width 0.25) (layer "F.Cu") (net 8))
+  (via (at 126.5 85) (size 0.8) (drill 0.4) (layers "F.Cu" "B.Cu") (net 8))
+  (segment (start 126.5 85) (end 124.945 83.445) (width 0.25) (layer "B.Cu") (net 8))
+  (segment (start 124.945 83.445) (end 119.675 83.445) (width 0.25) (layer "B.Cu") (net 8))
   (segment (start 119.675 83.445) (end 118.5 84.62) (width 0.25) (layer "B.Cu") (net 8))
-  (segment (start 125.445 83.445) (end 119.675 83.445) (width 0.25) (layer "B.Cu") (net 8))
-  (segment (start 126.5 84.5) (end 125.445 83.445) (width 0.25) (layer "B.Cu") (net 8))
   (segment (start 123.5 79.46) (end 121.04 77) (width 0.25) (layer "F.Cu") (net 9))
   (segment (start 123.717001 84.927499) (end 123.5 84.710498) (width 0.25) (layer "F.Cu") (net 9))
@@
   (segment (start 124.7869 78.2131) (end 126 77) (width 0.25) (layer "F.Cu") (net 20))
   (segment (start 124.7869 80.377501) (end 124.7869 78.2131) (width 0.25) (layer "F.Cu") (net 20))
+  (segment (start 126.236593 80.738102) (end 125.947195 81.0275) (width 0.25) (layer "F.Cu") (net 21))
+  (segment (start 128.738102 80.738102) (end 126.236593 80.738102) (width 0.25) (layer "F.Cu") (net 21))
+  (segment (start 125.947195 81.0275) (end 124.7869 81.0275) (width 0.25) (layer "F.Cu") (net 21))
+  (segment (start 129.275 81.275) (end 128.738102 80.738102) (width 0.25) (layer "F.Cu") (net 21))
+  (segment (start 129.275 86.775) (end 129.275 81.275) (width 0.25) (layer "F.Cu") (net 21))
+  (segment (start 130.5 88) (end 129.275 86.775) (width 0.25) (layer "F.Cu") (net 21))
+  (via (at 130.5 88) (size 0.8) (drill 0.4) (layers "F.Cu" "B.Cu") (net 21))
+  (segment (start 128.825 90.825) (end 128.825 82.725901) (width 0.25) (layer "F.Cu") (net 22))
+  (segment (start 125.824092 81.786999) (end 125.213001 81.786999) (width 0.25) (layer "F.Cu") (net 22))
+  (segment (start 130.5 92.5) (end 128.825 90.825) (width 0.25) (layer "F.Cu") (net 22))
+  (segment (start 127.338839 81.23974) (end 126.371351 81.23974) (width 0.25) (layer "F.Cu") (net 22))
+  (segment (start 128.825 82.725901) (end 127.338839 81.23974) (width 0.25) (layer "F.Cu") (net 22))
+  (segment (start 126.371351 81.23974) (end 125.824092 81.786999) (width 0.25) (layer "F.Cu") (net 22))
+  (via (at 130.5 92.5) (size 0.8) (drill 0.4) (layers "F.Cu" "B.Cu") (net 22))
   (segment (start 122.665 84.525497) (end 122.665 81.165) (width 0.25) (layer "F.Cu") (net 23))
   (segment (start 123.717001 85.577498) (end 122.665 84.525497) (width 0.25) (layer "F.Cu") (net 23))
   (segment (start 124.7869 85.577498) (end 123.717001 85.577498) (width 0.25) (layer "F.Cu") (net 23))
   (segment (start 122.665 81.165) (end 121.04 79.54) (width 0.25) (layer "F.Cu") (net 23))
+  (segment (start 132.0513 82.327502) (end 130.981401 82.327502) (width 0.25) (layer "F.Cu") (net 24))
+  (segment (start 130.5 82.808903) (end 130.5 84) (width 0.25) (layer "F.Cu") (net 24))
+  (segment (start 130.981401 82.327502) (end 130.5 82.808903) (width 0.25) (layer "F.Cu") (net 24))
+  (via (at 130.5 84) (size 0.8) (drill 0.4) (layers "F.Cu" "B.Cu") (net 24))
   (zone (net 4) (net_name "GND") (layers F&B.Cu) (hatch edge 0.508)
     (connect_pads yes (clearance 0.508))
