File: PCA9535/PCA9535.kicad_pcb (KiCad board)
At the start: 2 copper layers, 25 x 25 mm, 16 parts, among them J1 Conn_01x04, J2 Conn_01x04, J3 Conn_02x05_Odd_Even, J4 Conn_01x01, J6 Conn_02x05_Odd_Even, U1 PCA9535

Commit message: Finalizing the 16pin expander
Parts:
- U1: value PCA9535 -> PCA9535DBR
Routing:
- net P03: track 11.1 -> 12.4 mm
- net GND: vias 2 -> 4
Changed lines of the file:
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@@
       (effects (font (size 1 1) (thickness 0.15)))
     )
-    (fp_text value "PCA9535" (at 0 5.5475) (layer "F.SilkS")
+    (fp_text value "PCA9535DBR" (at 0 5.5475) (layer "F.SilkS")
       (effects (font (size 1 1) (thickness 0.15)))
     )
@@
       (net 24 "A0") (pinfunction "A0") (pintype "input"))
     (pad "22" smd rect (at 3.6322 -2.274999) (size 1.639799 0.431) (layers "F.Cu" "F.Paste" "F.Mask")
-      (net 3 "SCL") (pinfunction "SCL") (pintype "unspecified"))
+      (net 3 "SCL") (pinfunction "SCL") (pintype "input"))
     (pad "23" smd rect (at 3.6322 -2.924998) (size 1.639799 0.431) (layers "F.Cu" "F.Paste" "F.Mask")
-      (net 2 "SDA") (pinfunction "SDA") (pintype "unspecified"))
+      (net 2 "SDA") (pinfunction "SDA") (pintype "bidirectional"))
     (pad "24" smd rect (at 3.6322 -3.574999) (size 1.639799 0.431) (layers "F.Cu" "F.Paste" "F.Mask")
       (net 1 "+3.3V") (pinfunction "VCC") (pintype "power_in"))
@@
     (property "Sheetname" "")
     (attr smd)
-    (fp_text reference "R1" (at -2.5 0) (layer "F.SilkS")
-      (effects (font (size 0.5 0.5) (thickness 0.125)))
+    (fp_text reference "R1" (at 0 0) (layer "F.SilkS")
+      (effects (font (size 0.4 0.4) (thickness 0.1)))
     )
     (fp_text value "4.7k" (at 0 1.65) (layer "F.Fab") hide
@@
     (property "Sheetname" "")
     (attr smd)
-    (fp_text reference "R2" (at -2.5 0) (layer "F.SilkS")
-      (effects (font (size 0.5 0.5) (thickness 0.125)))
+    (fp_text reference "R2" (at 0 0) (layer "F.SilkS")
+      (effects (font (size 0.4 0.4) (thickness 0.1)))
     )
     (fp_text value "4.7k" (at 0 1.65) (layer "F.Fab") hide
@@
     (property "Sheetname" "")
     (attr smd)
-    (fp_text reference "R3" (at -2.5 0) (layer "F.SilkS")
-      (effects (font (size 0.5 0.5) (thickness 0.125)))
+    (fp_text reference "R3" (at 0 0) (layer "F.SilkS")
+      (effects (font (size 0.4 0.4) (thickness 0.1)))
     )
     (fp_text value "4.7k" (at 0 1.65) (layer "F.Fab") hide
@@
   )
   (gr_rect (start 116.5 69.5) (end 141.5 94.5) (layer "Edge.Cuts") (width 0.1) (fill none))
-  (gr_text "gnd" (at 127.5 92.5 90) (layer "B.Cu")
+  (gr_text "gnd" (at 127.5 92.5 90) (layer "B.SilkS")
     (effects (font (size 0.5 0.5) (thickness 0.125)) (justify mirror))
   )
-  (gr_text "3V3" (at 133.5 84.5) (layer "B.Cu")
+  (gr_text "3V3" (at 133.5 84.5) (layer "B.SilkS")
     (effects (font (size 0.5 0.5) (thickness 0.125)) (justify mirror))
   )
-  (gr_text "gnd" (at 127.5 84.5 90) (layer "B.Cu")
+  (gr_text "gnd" (at 127.5 84.5 90) (layer "B.SilkS")
     (effects (font (size 0.5 0.5) (thickness 0.125)) (justify mirror))
   )
-  (gr_text "gnd" (at 127.5 88.5 90) (layer "B.Cu")
+  (gr_text "gnd" (at 127.5 88.5 90) (layer "B.SilkS")
     (effects (font (size 0.5 0.5) (thickness 0.125)) (justify mirror))
   )
-  (gr_text "3V3" (at 133.5 92.5) (layer "B.Cu")
+  (gr_text "3V3" (at 133.5 92.5) (layer "B.SilkS")
     (effects (font (size 0.5 0.5) (thickness 0.125)) (justify mirror))
   )
-  (gr_text "3V3" (at 133.5 88.5) (layer "B.Cu")
+  (gr_text "3V3" (at 133.5 88.5) (layer "B.SilkS")
     (effects (font (size 0.5 0.5) (thickness 0.125)) (justify mirror))
   )
@@
     (effects (font (size 0.5 0.5) (thickness 0.125)))
   )
-  (gr_text "3v3" (at 140 75) (layer "F.SilkS")
+  (gr_text "3v3" (at 140 74.676) (layer "F.SilkS")
     (effects (font (size 1 1) (thickness 0.15)))
   )
-  (gr_text "GND" (at 137 75) (layer "F.SilkS")
+  (gr_text "GND" (at 137 74.676) (layer "F.SilkS")
     (effects (font (size 1 1) (thickness 0.15)))
   )
@@
   (segment (start 130 73.5) (end 132 75.5) (width 0.25) (layer "B.Cu") (net 3))
   (via (at 131.5 73.5) (size 0.8) (drill 0.4) (layers "F.Cu" "B.Cu") (net 4))
+  (via (at 121.666 91.948) (size 0.8) (drill 0.4) (layers "F.Cu" "B.Cu") (free) (net 4))
+  (via (at 132.842 90.678) (size 0.8) (drill 0.4) (layers "F.Cu" "B.Cu") (free) (net 4))
   (via (at 123.5 73.5) (size 0.8) (drill 0.4) (layers "F.Cu" "B.Cu") (net 4))
   (segment (start 127.038534 81.96474) (end 126.675775 82.327499) (width 0.25) (layer "F.Cu") (net 5))
@@
   (segment (start 127.084386 83.03519) (end 122.414196 78.365) (width 0.25) (layer "B.Cu") (net 6))
   (segment (start 122.414196 78.365) (end 119.675 78.365) (width 0.25) (layer "B.Cu") (net 6))
-  (segment (start 126.825205 84.054883) (end 126.397821 83.627499) (width 0.25) (layer "F.Cu") (net 7))
-  (segment (start 126.397821 83.627499) (end 124.7869 83.627499) (width 0.25) (layer "F.Cu") (net 7))
-  (via (at 126.825205 84.054883) (size 0.8) (drill 0.4) (layers "F.Cu" "B.Cu") (net 7))
-  (segment (start 126.825205 83.800607) (end 123.929598 80.905) (width 0.25) (layer "B.Cu") (net 7))
+  (segment (start 126.732512 84.34607) (end 126.013941 83.627499) (width 0.25) (layer "F.Cu") (net 7))
+  (segment (start 126.013941 83.627499) (end 124.7869 83.627499) (width 0.25) (layer "F.Cu") (net 7))
+  (via (at 126.732512 84.34607) (size 0.8) (drill 0.4) (layers "F.Cu" "B.Cu") (net 7))
+  (segment (start 119.675 80.905) (end 118.5 82.08) (width 0.25) (layer "B.Cu") (net 7))
+  (segment (start 126.732512 83.707914) (end 123.929598 80.905) (width 0.25) (layer "B.Cu") (net 7))
+  (segment (start 126.732512 84.34607) (end 126.732512 83.707914) (width 0.25) (layer "B.Cu") (net 7))
   (segment (start 123.929598 80.905) (end 119.675 80.905) (width 0.25) (layer "B.Cu") (net 7))
-  (segment (start 126.825205 84.054883) (end 126.825205 83.800607) (width 0.25) (layer "B.Cu") (net 7))
-  (segment (start 119.675 80.905) (end 118.5 82.08) (width 0.25) (layer "B.Cu") (net 7))
-  (segment (start 126.5 85) (end 125.777498 84.277498) (width 0.25) (layer "F.Cu") (net 8))
-  (segment (start 125.777498 84.277498) (end 124.7869 84.277498) (width 0.25) (layer "F.Cu") (net 8))
-  (via (at 126.5 85) (size 0.8) (drill 0.4) (layers "F.Cu" "B.Cu") (net 8))
-  (segment (start 126.5 85) (end 124.945 83.445) (width 0.25) (layer "B.Cu") (net 8))
-  (segment (start 124.945 83.445) (end 119.675 83.445) (width 0.25) (layer "B.Cu") (net 8))
+  (segment (start 126.5 85.352) (end 125.931799 84.783799) (width 0.25) (layer "F.Cu") (net 8))
+  (segment (start 126.5 85.852) (end 126.5 85.352) (width 0.25) (layer "F.Cu") (net 8))
+  (segment (start 125.931799 84.783799) (end 125.931799 84.386999) (width 0.25) (layer "F.Cu") (net 8))
+  (segment (start 125.931799 84.386999) (end 125.822298 84.277498) (width 0.25) (layer "F.Cu") (net 8))
+  (segment (start 125.822298 84.277498) (end 124.7869 84.277498) (width 0.25) (layer "F.Cu") (net 8))
+  (via (at 126.5 85.852) (size 0.8) (drill 0.4) (layers "F.Cu" "B.Cu") (net 8))
+  (segment (start 126.5 85.852) (end 124.093 83.445) (width 0.25) (layer "B.Cu") (net 8))
+  (segment (start 124.093 83.445) (end 119.675 83.445) (width 0.25) (layer "B.Cu") (net 8))
   (segment (start 119.675 83.445) (end 118.5 84.62) (width 0.25) (layer "B.Cu") (net 8))
   (segment (start 123.5 79.46) (end 121.04 77) (width 0.25) (layer "F.Cu") (net 9))

Commit message: syncing
Parts:
- J1, J2: footprint Connector_JST:JST_SH_BM04B-SRSS-TB_1x04-1MP_P1.00mm_Vertical -> Connector_JST:JST_SH_SM04B-SRSS-TB_1x04-1MP_P1.00mm_Horizontal
- moved R3 41.9 mm to (166.5, 82.5)
- moved J1 41.8 mm to (174.5, 77.0), turned to 180 degrees
- moved J2 41.8 mm to (166.5, 77.0), turned to 180 degrees
- moved J4 41.8 mm to (170.5, 82.0)
- moved R1 41.8 mm to (174.5, 83.0)
- moved R2 41.8 mm to (174.5, 81.0)
- moved H1 41.7 mm to (160.0, 76.0)
- moved H2 41.7 mm to (181.0, 76.0)
- moved H3 41.7 mm to (181.0, 97.0)
- moved H4 41.7 mm to (160.0, 97.0)
- moved J3 41.7 mm to (160.0, 81.5)
- moved J6 41.7 mm to (181.5, 91.5)
- moved JP1 41.7 mm to (172.0, 89.0)
- moved JP2 41.7 mm to (172.0, 93.0)
- moved JP3 41.7 mm to (172.0, 97.0)
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Routing:
- net +3.3V: track 90.3 -> 75.9 mm
- net SCL: track 18.5 -> 23.7 mm, vias 4 -> 3
- net INT: track 6.88 -> 6.29 mm
- net GND: vias 4 -> 3
