File: Template/Template.kicad_pcb (KiCad board)
At the start: 2 copper layers, 25 x 25 mm, 16 parts, among them J1 Conn_01x04, J2 Conn_01x04, J3 Conn_02x05_Odd_Even, J4 Conn_01x01, J6 Conn_02x05_Odd_Even, U1 PCA9535

Commit message: Futher Progress on the gpio
Parts:
- U1: value PCA9535 -> PCA9535DBR
Routing:
- net GND: vias 2 -> 3
Other:
- board text removed: "00"
- board text removed: "10"
- board text removed: "3V3"
- board text removed: "Bank 0"
- board text removed: "Bank 1"
- board text removed: "gnd"
Changed lines of the file:
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@@
       (outputformat 1)
       (mirror false)
-      (drillshape 0)
+      (drillshape 1)
       (scaleselection 1)
-      (outputdirectory "Gerbers/")
+      (outputdirectory "")
     )
   )
@@
       (effects (font (size 1 1) (thickness 0.15)))
     )
-    (fp_text value "PCA9535" (at 0 5.5475) (layer "F.SilkS")
+    (fp_text value "PCA9535DBR" (at 0 8.5475) (layer "F.SilkS")
       (effects (font (size 1 1) (thickness 0.15)))
     )
@@
     (pad "4" smd roundrect (at 1.5 1.325) (size 0.6 1.55) (layers "F.Cu" "F.Paste" "F.Mask") (roundrect_rratio 0.25)
       (net 3 "SCL") (pinfunction "Pin_4") (pintype "passive"))
-    (pad "MP" smd roundrect (at -2.8 -1.2) (size 1.2 1.8) (layers "F.Cu" "F.Paste" "F.Mask") (roundrect_rratio 0.2083333333))
-    (pad "MP" smd roundrect (at 2.8 -1.2) (size 1.2 1.8) (layers "F.Cu" "F.Paste" "F.Mask") (roundrect_rratio 0.2083333333))
+    (pad "MP" smd roundrect (at -2.8 -1.2) (size 1.2 1.8) (layers "F.Cu" "F.Paste" "F.Mask") (roundrect_rratio 0.208333))
+    (pad "MP" smd roundrect (at 2.8 -1.2) (size 1.2 1.8) (layers "F.Cu" "F.Paste" "F.Mask") (roundrect_rratio 0.208333))
     (model "${KICAD6_3DMODEL_DIR}/Connector_JST.3dshapes/JST_SH_BM04B-SRSS-TB_1x04-1MP_P1.00mm_Vertical.wrl"
       (offset (xyz 0 0 0))
@@
     (fp_line (start 1 0.625) (end -1 0.625) (layer "F.Fab") (width 0.1))
     (fp_line (start -1 0.625) (end -1 -0.625) (layer "F.Fab") (width 0.1))
-    (pad "1" smd roundrect (at -1 0 180) (size 1.2 1.4) (layers "F.Cu" "F.Paste" "F.Mask") (roundrect_rratio 0.2083333333)
+    (pad "1" smd roundrect (at -1 0 180) (size 1.2 1.4) (layers "F.Cu" "F.Paste" "F.Mask") (roundrect_rratio 0.208333)
       (net 1 "+3.3V") (pintype "passive"))
-    (pad "2" smd roundrect (at 1 0 180) (size 1.2 1.4) (layers "F.Cu" "F.Paste" "F.Mask") (roundrect_rratio 0.2083333333)
+    (pad "2" smd roundrect (at 1 0 180) (size 1.2 1.4) (layers "F.Cu" "F.Paste" "F.Mask") (roundrect_rratio 0.208333)
       (net 3 "SCL") (pintype "passive"))
     (model "${KICAD6_3DMODEL_DIR}/Resistor_SMD.3dshapes/R_0805_2012Metric.wrl"
@@
     (fp_line (start 1 0.625) (end -1 0.625) (layer "F.Fab") (width 0.1))
     (fp_line (start -1 -0.625) (end 1 -0.625) (layer "F.Fab") (width 0.1))
-    (pad "1" smd roundrect (at -1 0 180) (size 1.2 1.4) (layers "F.Cu" "F.Paste" "F.Mask") (roundrect_rratio 0.2083333333)
+    (pad "1" smd roundrect (at -1 0 180) (size 1.2 1.4) (layers "F.Cu" "F.Paste" "F.Mask") (roundrect_rratio 0.208333)
       (net 1 "+3.3V") (pintype "passive"))
-    (pad "2" smd roundrect (at 1 0 180) (size 1.2 1.4) (layers "F.Cu" "F.Paste" "F.Mask") (roundrect_rratio 0.2083333333)
+    (pad "2" smd roundrect (at 1 0 180) (size 1.2 1.4) (layers "F.Cu" "F.Paste" "F.Mask") (roundrect_rratio 0.208333)
       (net 2 "SDA") (pintype "passive"))
     (model "${KICAD6_3DMODEL_DIR}/Resistor_SMD.3dshapes/R_0805_2012Metric.wrl"
@@
     (property "Sheetname" "")
     (attr through_hole)
-    (fp_text reference "J6" (at 1.27 -2.33) (layer "F.SilkS") hide
+    (fp_text reference "J6" (at 1.27 -2.33) (layer "F.SilkS")
       (effects (font (size 1 1) (thickness 0.15)))
     )
@@
     (pad "4" smd roundrect (at 1.5 1.325) (size 0.6 1.55) (layers "F.Cu" "F.Paste" "F.Mask") (roundrect_rratio 0.25)
       (net 3 "SCL") (pinfunction "Pin_4") (pintype "passive"))
-    (pad "MP" smd roundrect (at -2.8 -1.2) (size 1.2 1.8) (layers "F.Cu" "F.Paste" "F.Mask") (roundrect_rratio 0.2083333333))
-    (pad "MP" smd roundrect (at 2.8 -1.2) (size 1.2 1.8) (layers "F.Cu" "F.Paste" "F.Mask") (roundrect_rratio 0.2083333333))
+    (pad "MP" smd roundrect (at -2.8 -1.2) (size 1.2 1.8) (layers "F.Cu" "F.Paste" "F.Mask") (roundrect_rratio 0.208333))
+    (pad "MP" smd roundrect (at 2.8 -1.2) (size 1.2 1.8) (layers "F.Cu" "F.Paste" "F.Mask") (roundrect_rratio 0.208333))
     (model "${KICAD6_3DMODEL_DIR}/Connector_JST.3dshapes/JST_SH_BM04B-SRSS-TB_1x04-1MP_P1.00mm_Vertical.wrl"
       (offset (xyz 0 0 0))
@@
     (property "Sheetname" "")
     (attr through_hole)
-    (fp_text reference "J3" (at 1.27 -2.33) (layer "F.SilkS") hide
+    (fp_text reference "J3" (at 1.27 -2.33) (layer "F.SilkS")
       (effects (font (size 1 1) (thickness 0.15)))
     )
@@
     (fp_line (start 1 -0.625) (end 1 0.625) (layer "F.Fab") (width 0.1))
     (fp_line (start -1 0.625) (end -1 -0.625) (layer "F.Fab") (width 0.1))
-    (pad "1" smd roundrect (at -1 0) (size 1.2 1.4) (layers "F.Cu" "F.Paste" "F.Mask") (roundrect_rratio 0.2083333333)
+    (pad "1" smd roundrect (at -1 0) (size 1.2 1.4) (layers "F.Cu" "F.Paste" "F.Mask") (roundrect_rratio 0.208333)
       (net 1 "+3.3V") (pintype "passive"))
-    (pad "2" smd roundrect (at 1 0) (size 1.2 1.4) (layers "F.Cu" "F.Paste" "F.Mask") (roundrect_rratio 0.2083333333)
+    (pad "2" smd roundrect (at 1 0) (size 1.2 1.4) (layers "F.Cu" "F.Paste" "F.Mask") (roundrect_rratio 0.208333)
       (net 20 "INT") (pintype "passive"))
     (model "${KICAD6_3DMODEL_DIR}/Resistor_SMD.3dshapes/R_0805_2012Metric.wrl"
@@
       (effects (font (size 1 1) (thickness 0.15)) (justify mirror))
     )
-    (fp_text value "SolderJumper_3_Open" (at 0 -2) (layer "B.Fab") hide
+    (fp_text value "SolderJumper_3_Open" (at 0 -2) (layer "B.Fab")
       (effects (font (size 1 1) (thickness 0.15)) (justify mirror))
     )
@@
       (effects (font (size 1 1) (thickness 0.15)) (justify mirror))
     )
-    (fp_text value "SolderJumper_3_Open" (at 0 -2) (layer "B.Fab") hide
+    (fp_text value "SolderJumper_3_Open" (at 0 -2) (layer "B.Fab")
       (effects (font (size 1 1) (thickness 0.15)) (justify mirror))
     )
@@
   )
   (gr_rect (start 116.5 69.5) (end 141.5 94.5) (layer "Edge.Cuts") (width 0.1) (fill none))
-  (gr_text "gnd" (at 127.5 92.5 90) (layer "B.Cu")
-    (effects (font (size 0.5 0.5) (thickness 0.125)) (justify mirror))
-  )
-  (gr_text "3V3" (at 133.5 84.5) (layer "B.Cu")
-    (effects (font (size 0.5 0.5) (thickness 0.125)) (justify mirror))
-  )
-  (gr_text "gnd" (at 127.5 84.5 90) (layer "B.Cu")
-    (effects (font (size 0.5 0.5) (thickness 0.125)) (justify mirror))
-  )
-  (gr_text "gnd" (at 127.5 88.5 90) (layer "B.Cu")
-    (effects (font (size 0.5 0.5) (thickness 0.125)) (justify mirror))
-  )
-  (gr_text "3V3" (at 133.5 92.5) (layer "B.Cu")
-    (effects (font (size 0.5 0.5) (thickness 0.125)) (justify mirror))
-  )
-  (gr_text "3V3" (at 133.5 88.5) (layer "B.Cu")
-    (effects (font (size 0.5 0.5) (thickness 0.125)) (justify mirror))
-  )
   (gr_text "GND" (at 121 89.5) (layer "F.SilkS")
     (effects (font (size 1 1) (thickness 0.15)))
   )
-  (gr_text "10" (at 140 89) (layer "F.SilkS")
-    (effects (font (size 0.5 0.5) (thickness 0.125)))
-  )
   (gr_text "3v3" (at 140 75) (layer "F.SilkS")
     (effects (font (size 1 1) (thickness 0.15)))
@@
     (effects (font (size 1 1) (thickness 0.15)))
   )
-  (gr_text "Bank 1" (at 137 89) (layer "F.SilkS")
-    (effects (font (size 0.4 0.4) (thickness 0.1)))
-  )
-  (gr_text "Designed by Fortinbra\nfortinbra@becauseimclever.com" (at 129 92.5) (layer "F.SilkS")
+  (gr_text "Designed by Fortinbra\nfortinbra@becauseimclever.com" (at 129 90) (layer "F.SilkS")
     (effects (font (size 0.75 0.75) (thickness 0.05)))
-  )
-  (gr_text "00" (at 118.5 75) (layer "F.SilkS")
-    (effects (font (size 0.5 0.5) (thickness 0.125)))
   )
   (gr_text "3v3" (at 118 89.5) (layer "F.SilkS")
     (effects (font (size 1 1) (thickness 0.15)))
-  )
-  (gr_text "Bank 0" (at 121.5 75) (layer "F.SilkS")
-    (effects (font (size 0.4 0.4) (thickness 0.1)))
   )
   (segment (start 133.353249 72.025) (end 134.646751 72.025) (width 0.25) (layer "F.Cu") (net 1))
@@
   (segment (start 128.5 73.5) (end 130 73.5) (width 0.25) (layer "B.Cu") (net 3))
   (segment (start 130 73.5) (end 132 75.5) (width 0.25) (layer "B.Cu") (net 3))
+  (via (at 127.5 92.5) (size 0.8) (drill 0.4) (layers "F.Cu" "B.Cu") (free) (net 4))
   (via (at 131.5 73.5) (size 0.8) (drill 0.4) (layers "F.Cu" "B.Cu") (net 4))
   (via (at 123.5 73.5) (size 0.8) (drill 0.4) (layers "F.Cu" "B.Cu") (net 4))
