File: TCA9534/TCA9534.kicad_pcb (KiCad board)
At the start: 2 copper layers, 25 x 25 mm, 14 parts, among them J1 Conn_01x04, J2 Conn_01x04, J3 Conn_02x05_Odd_Even, U1 TCA9534

Commit message: SYNC
Parts:
- added J4: Conn_01x01, Connector_PinHeader_2.54mm:PinHeader_1x01_P2.54mm_Vertical, F.Cu at (179.0, 89.0)
Routing:
- net /INT: track 3.53 -> 6.53 mm
Changed lines of the file:
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@@
     (property "Sheetname" "")
     (attr exclude_from_pos_files)
-    (fp_text reference "H2" (at 0 -3.5) (layer "F.SilkS")
+    (fp_text reference "H2" (at 0 -3.5) (layer "F.SilkS") hide
       (effects (font (size 1 1) (thickness 0.15)))
     )
@@
     (property "Sheetname" "")
     (attr through_hole)
-    (fp_text reference "U1" (at 0 -2.54) (layer "F.SilkS")
-      (effects (font (size 1 1) (thickness 0.15)))
-    )
-    (fp_text value "TCA9534" (at 0 0) (layer "F.SilkS")
+    (fp_text reference "U1" (at 0 -4) (layer "F.SilkS")
+      (effects (font (size 1 1) (thickness 0.15)))
+    )
+    (fp_text value "TCA9534" (at 0 -2) (layer "F.SilkS")
       (effects (font (size 1 1) (thickness 0.15)))
     )
@@
       (net 2 "+3.3V") (pinfunction "VCC") (pintype "power_in"))
   )
+  (footprint "Connector_PinHeader_2.54mm:PinHeader_1x01_P2.54mm_Vertical" (layer "F.Cu")
+    (at 179 89)
+    (descr "Through hole straight pin header, 1x01, 2.54mm pitch, single row")
+    (tags "Through hole pin header THT 1x01 2.54mm single row")
+    (property "Sheetfile" "TCA9534.kicad_sch")
+    (property "Sheetname" "")
+    (attr through_hole)
+    (fp_text reference "J4" (at 0 -2.33) (layer "F.SilkS") hide
+      (effects (font (size 1 1) (thickness 0.15)))
+    )
+    (fp_text value "Conn_01x01" (at 0 2.33) (layer "F.Fab")
+      (effects (font (size 1 1) (thickness 0.15)))
+    )
+    (fp_text user "INT" (at 0 2 unlocked) (layer "F.SilkS")
+      (effects (font (size 0.75 0.75) (thickness 0.15)))
+    )
+    (fp_text user "${REFERENCE}" (at 0 0 90) (layer "F.Fab")
+      (effects (font (size 1 1) (thickness 0.15)))
+    )
+    (fp_line (start -1.33 1.27) (end -1.33 1.33) (layer "F.SilkS") (width 0.12))
+    (fp_line (start -1.33 0) (end -1.33 -1.33) (layer "F.SilkS") (width 0.12))
+    (fp_line (start 1.33 1.27) (end 1.33 1.33) (layer "F.SilkS") (width 0.12))
+    (fp_line (start -1.33 -1.33) (end 0 -1.33) (layer "F.SilkS") (width 0.12))
+    (fp_line (start -1.33 1.27) (end 1.33 1.27) (layer "F.SilkS") (width 0.12))
+    (fp_line (start -1.33 1.33) (end 1.33 1.33) (layer "F.SilkS") (width 0.12))
+    (fp_line (start 1.8 1.8) (end 1.8 -1.8) (layer "F.CrtYd") (width 0.05))
+    (fp_line (start 1.8 -1.8) (end -1.8 -1.8) (layer "F.CrtYd") (width 0.05))
+    (fp_line (start -1.8 -1.8) (end -1.8 1.8) (layer "F.CrtYd") (width 0.05))
+    (fp_line (start -1.8 1.8) (end 1.8 1.8) (layer "F.CrtYd") (width 0.05))
+    (fp_line (start 1.27 1.27) (end -1.27 1.27) (layer "F.Fab") (width 0.1))
+    (fp_line (start -1.27 1.27) (end -1.27 -0.635) (layer "F.Fab") (width 0.1))
+    (fp_line (start -1.27 -0.635) (end -0.635 -1.27) (layer "F.Fab") (width 0.1))
+    (fp_line (start 1.27 -1.27) (end 1.27 1.27) (layer "F.Fab") (width 0.1))
+    (fp_line (start -0.635 -1.27) (end 1.27 -1.27) (layer "F.Fab") (width 0.1))
+    (pad "1" thru_hole rect (at 0 0) (size 1.7 1.7) (drill 1) (layers *.Cu *.Mask)
+      (net 16 "/INT") (pinfunction "Pin_1") (pintype "passive"))
+    (model "${KICAD6_3DMODEL_DIR}/Connector_PinHeader_2.54mm.3dshapes/PinHeader_1x01_P2.54mm_Vertical.wrl"
+      (offset (xyz 0 0 0))
+      (scale (xyz 1 1 1))
+      (rotate (xyz 0 0 0))
+    )
+  )
   (footprint "Jumper:SolderJumper-3_P1.3mm_Open_Pad1.0x1.5mm" (layer "F.Cu")
     (at 161 90)
@@
     (property "Sheetname" "")
     (attr exclude_from_pos_files)
-    (fp_text reference "H1" (at 0 -3.5) (layer "F.SilkS")
+    (fp_text reference "H1" (at 0 -3.5) (layer "F.SilkS") hide
       (effects (font (size 1 1) (thickness 0.15)))
     )
@@
     (property "Sheetname" "")
     (attr exclude_from_pos_files)
-    (fp_text reference "H4" (at 0 -3.5) (layer "F.SilkS")
+    (fp_text reference "H4" (at 0 -3.5) (layer "F.SilkS") hide
       (effects (font (size 1 1) (thickness 0.15)))
     )
@@
   (segment (start 161 90) (end 161 89.2) (width 0.25) (layer "F.Cu") (net 15))
   (segment (start 178.365 85.365) (end 175.7371 85.365) (width 0.25) (layer "F.Cu") (net 16))
+  (segment (start 179 86) (end 179 89) (width 0.25) (layer "F.Cu") (net 16))
   (segment (start 179 86) (end 178.365 85.365) (width 0.25) (layer "F.Cu") (net 16))
   (zone (net 1) (net_name "GND") (layers F&B.Cu) (hatch edge 0.508)
