File: TCA9534/TCA9534.kicad_sch (KiCad schematic)
At the start: 14 parts, among them J1 Conn_01x04, J2 Conn_01x04, J3 Conn_02x05_Odd_Even, U1 TCA9534DWR

Commit message: SYNC
Parts:
- added J4: Conn_01x01, symbol Connector_Generic:Conn_01x01
- JP1, JP2, JP3: footprint (none) -> Jumper:SolderJumper-3_P1.3mm_Open_Pad1.0x1.5mm
Connections:
- net INT: now also J4.1 (Pin_1)
Changed lines of the file:
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@@
+    (effects (font (size 1.27 1.27)) (justify right bottom))
+  )
+  (label "INT" (at 67.31 101.6 180)
     (effects (font (size 1.27 1.27)) (justify right bottom))
   )
@@
     (property "Reference" "JP2" (id 0) (at 90.17 34.29 0))
     (property "Value" "SolderJumper_3_Open" (id 1) (at 90.17 36.83 0))
-    (property "Footprint" "" (id 2) (at 90.17 40.64 0)
+    (property "Footprint" "Jumper:SolderJumper-3_P1.3mm_Open_Pad1.0x1.5mm" (id 2) (at 90.17 40.64 0)
       (effects (font (size 1.27 1.27)) hide)
     )
@@
     (property "Reference" "JP1" (id 0) (at 90.17 17.78 0))
     (property "Value" "SolderJumper_3_Open" (id 1) (at 90.17 20.32 0))
-    (property "Footprint" "" (id 2) (at 90.17 24.13 0)
+    (property "Footprint" "Jumper:SolderJumper-3_P1.3mm_Open_Pad1.0x1.5mm" (id 2) (at 90.17 24.13 0)
       (effects (font (size 1.27 1.27)) hide)
     )
@@
     (pin "4")
   )
+  (symbol (lib_id "Connector_Generic:Conn_01x01") (at 72.39 101.6 0) (unit 1)
+    (in_bom yes) (on_board yes) (fields_autoplaced)
+    (property "Reference" "J4" (id 0) (at 74.93 100.3299 0)
+      (effects (font (size 1.27 1.27)) (justify left))
+    )
+    (property "Value" "Conn_01x01" (id 1) (at 74.93 102.8699 0)
+      (effects (font (size 1.27 1.27)) (justify left))
+    )
+    (property "Footprint" "" (id 2) (at 72.39 101.6 0)
+      (effects (font (size 1.27 1.27)) hide)
+    )
+    (property "Datasheet" "~" (id 3) (at 72.39 101.6 0)
+      (effects (font (size 1.27 1.27)) hide)
+    )
+    (pin "1")
+  )
   (symbol (lib_id "power:GND") (at 99.06 40.64 0) (unit 1)
     (in_bom yes) (on_board yes) (fields_autoplaced)
@@
     (property "Reference" "JP3" (id 0) (at 90.17 50.8 0))
     (property "Value" "SolderJumper_3_Open" (id 1) (at 90.17 53.34 0))
-    (property "Footprint" "" (id 2) (at 90.17 57.15 0)
+    (property "Footprint" "Jumper:SolderJumper-3_P1.3mm_Open_Pad1.0x1.5mm" (id 2) (at 90.17 57.15 0)
       (effects (font (size 1.27 1.27)) hide)
     )
@@
       (reference "J3") (unit 1) (value "Conn_02x05_Odd_Even") (footprint "Connector_PinHeader_2.54mm:PinHeader_2x05_P2.54mm_Vertical")
     )
+    (path "/2e28f08e-4e34-4cd0-af69-c0f135e21a70"
+      (reference "J4") (unit 1) (value "Conn_01x01") (footprint "Connector_PinHeader_2.54mm:PinHeader_1x01_P2.54mm_Vertical")
+    )
     (path "/1423e419-4831-4858-acd1-50db8803cee6"
